Commit message: STL in urdf, path change

File: diablo_plus/urdf/diablo_plus.urdf (robot description, URDF)
Before this commit: robot diablo_plus2, 7 links, 6 joints
Links:
- link base_link: geometry collision mesh filename=package://diablo_plus/meshes/base_link.STL; visual mesh filename=package://diablo_plus/meshes/base_link.STL
- link left_hip: geometry collision mesh filename=package://diablo_plus/meshes/left_hip.STL; visual mesh filename=package://diablo_plus/meshes/left_hip.STL
- link left_knee: geometry collision mesh filename=package://diablo_plus/meshes/left_knee.STL; visual mesh filename=package://diablo_plus/meshes/left_knee.STL
- link left_wheel: geometry collision mesh filename=package://diablo_plus/meshes/left_wheel.STL; visual mesh filename=package://diablo_plus/meshes/left_wheel.STL
- link right_hip: geometry collision mesh filename=package://diablo_plus/meshes/right_hip.STL; visual mesh filename=package://diablo_plus/meshes/right_hip.STL
- link right_knee: geometry collision mesh filename=package://diablo_plus/meshes/right_knee.STL; visual mesh filename=package://diablo_plus/meshes/right_knee.STL
- link right_wheel: geometry collision mesh filename=package://diablo_plus/meshes/right_wheel.STL; visual mesh filename=package://diablo_plus/meshes/right_wheel.STL

Commit message: diablo_plus urdf improve, try to fix

File: diablo_plus/urdf/diablo_plus.urdf (robot description, URDF)
Before this commit: robot diablo_plus2, 7 links, 6 joints
Joints:
- joint left_wheel_joint: limit effort=20 velocity=30 -> lower=0 upper=0 effort=20 velocity=30
- joint right_wheel_joint: limit effort=20 velocity=30 -> lower=0 upper=0 effort=20 velocity=30
